File: Hardware/electrical_diagram.sch (EAGLE design)
At the start: 103 parts, among them IC1 XC6220A331MR-G, IC2 BD5229G-TR, J1 112A-TAAR-R03_ATTEND, J2 SAMACSYS_PARTS_USB4110-GF-A, J3 FH34SRJ-24S-0.5SH_99_, J4 QWIIC_RIGHT_ANGLE, Q1 20V/4.2A/52mΩ/1.4W, Q2 SI1308EDL-T1-GE3, Q3 20V/4.2A/52mΩ/1.4W, U1 ESP32-C6-WROOM-1-N8, U2 MAX17048G+T10, U3 DS3231SN#, U4 W25Q512JVEIQ

Commit message: issues solved
Parts:
- removed TP10, TP13, TP14, TP15, TP16, TP17, TP2, TP3, TP4, TP5, TP9: TP, DeskAssistant v19 v1:TP
- added 3V3, EPD_3V3, EPD_3V3_C, EPD_BUSY, EPD_CS, GND, GND., INT_RTC, RX, VBAT, VBUS: TP, DeskAssistant v19 v1:TP
- CHG_LED: value (none) -> LED
- SJ1: value (none) -> -
- renumbered TP11 to EPD_DC, TP12 to EPD_RST, TP6 to MISO, TP7 to MOSI, TP8 to SCK
Connections:
- net 3V3: now also 3V3.TP; no longer TP16.TP
- net EPD_3V3: now also EPD_3V3.TP; no longer TP17.TP
- net EPD_3V3_C: now also EPD_3V3_C.TP; no longer TP13.TP
- net EPD_BUSY: now also EPD_BUSY.TP; no longer TP9.TP
- net EPD_CS: now also EPD_CS.TP; no longer TP10.TP
- net GND: now also GND..TP, GND.TP; no longer TP4.TP, TP5.TP
- net INT_RTC: now also INT_RTC.TP; no longer TP15.TP
- net RX: now also RX.TP; no longer TP2.TP
- net VBAT: now also VBAT.TP; no longer TP3.TP
- net VBUS: now also VBUS.TP; no longer TP14.TP
Other:
- moved on the sheet: C2, C4, D3, D4, D5, L1, Q2, R3, R4, R5, SJ1, TP1
