File: Hardware/electrical_diagram_pcb.brd (EAGLE design)
At the start: 200.7 x 117.4 mm, 103 parts, among them IC1 XC6220A331MR-G, IC2 BD5229G-TR, J1 112A-TAAR-R03_ATTEND, J2 SAMACSYS_PARTS_USB4110-GF-A, J3 FH34SRJ-24S-0.5SH_99_, J4 QWIIC_RIGHT_ANGLE, Q1 20V/4.2A/52mΩ/1.4W, Q2 SI1308EDL-T1-GE3, Q3 20V/4.2A/52mΩ/1.4W, U1 ESP32-C6-WROOM-1-N8, U2 MAX17048G+T10, U3 DS3231SN#, U4 W25Q512JVEIQ

Commit message: issues solved
Parts:
- removed TP12, TP6, TP7: TP, DeskAssistant v19 v1:TP20R
- added EPD_RST, MISO, MOSI: TP, DeskAssistant v19 v1:TP20R
- CHG_LED: value (none) -> LED
- SJ1: value (none) -> -
- moved C4 1.52 mm to (78.5, 0.09), turned to 90 degrees
- moved D10 1.39 mm to (39.4, 35.8), turned to 90 degrees
- moved C_DELAY 0.58 mm to (57.4, 77.5)
- renumbered TP10 to EPD_CS, TP11 to EPD_DC, TP13 to EPD_3V3_C, TP14 to VBUS, TP15 to INT_RTC, TP16 to 3V3, TP17 to EPD_3V3, TP2 to RX, TP3 to VBAT, TP4 to GND, TP5 to GND., TP8 to SCK, TP9 to EPD_BUSY
Connections:
- net EPD_RST: now also EPD_RST.TP; no longer TP12.TP
- net MISO: now also MISO.TP; no longer TP6.TP
- net MOSI: now also MOSI.TP; no longer TP7.TP
Routing:
- net GND: track 68.8 -> 34.2 mm, vias 21 -> 31
- net USB_D+: track 131.2 -> 147.3 mm
- net SRC: track 39.2 -> 51.5 mm, vias 3 -> 0
- net SCK: track 166.5 -> 176.2 mm, vias 5 -> 8
- net MOSI: track 149.3 -> 157.4 mm
- net 3V3: track 371.0 -> 378.8 mm
- net DP: track 21.2 -> 27.1 mm, vias 2 -> 0
- net RESET: track 97.4 -> 102.7 mm
- net DN: track 25.8 -> 30.2 mm
- net SS_SD: track 85.3 -> 89.4 mm, vias 3 -> 5
- net FLASH_CS: track 27.4 -> 31.4 mm, vias 4 -> 3
- net SDA: track 189.1 -> 185.2 mm
- net INT_RTC: track 89.7 -> 86.6 mm, vias 2 -> 4
- net N$7: track 19.9 -> 22.1 mm, vias 2 -> 3
- net EPD_RST: track 92.6 -> 94.6 mm, vias 2 -> 3
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Other:
- board size 200.7 x 117.4 mm -> 197.6 x 111.2 mm
